File: sample01.kicad_pcb (KiCad board)
At the start: 2 copper layers, 30.5 x 22.9 mm, 6 parts, among them J1 Power5V, Q1 2SC1815, SW1 SW_Push

Commit message: ベタグラウンド張り直し。ベタを張りなおしたので不要な配線削除。
Routing:
- net GND: track 146.1 -> 0.00 mm
Changed lines of the file:
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@@
     (thickness 1.6)
     (drawings 7)
-    (tracks 73)
+    (tracks 50)
     (zones 0)
     (modules 6)
@@
   (via (at 68.58 38.1) (size 0.8) (drill 0.4) (layers F.Cu B.Cu) (net 4))
   (via (at 68.58 35.56) (size 0.8) (drill 0.4) (layers F.Cu B.Cu) (net 4))
-  (segment (start 68.58 53.34) (end 68.58 50.8) (width 0.25) (layer B.Cu) (net 4))
-  (segment (start 68.58 50.8) (end 68.58 48.26) (width 0.25) (layer B.Cu) (net 4))
-  (segment (start 68.58 48.26) (end 68.58 38.1) (width 0.25) (layer B.Cu) (net 4))
-  (segment (start 68.58 38.1) (end 68.58 35.56) (width 0.25) (layer B.Cu) (net 4))
-  (segment (start 72.39 52.19) (end 72.39 53.34) (width 0.4) (layer B.Cu) (net 4))
-  (segment (start 79.999999 44.580001) (end 72.39 52.19) (width 0.4) (layer B.Cu) (net 4))
-  (segment (start 90.039999 44.580001) (end 79.999999 44.580001) (width 0.4) (layer B.Cu) (net 4))
-  (segment (start 93.98 40.64) (end 90.039999 44.580001) (width 0.4) (layer B.Cu) (net 4))
   (via (at 96.52 35.56) (size 0.8) (drill 0.4) (layers F.Cu B.Cu) (net 4))
   (via (at 93.98 35.56) (size 0.8) (drill 0.4) (layers F.Cu B.Cu) (net 4))
@@
   (via (at 96.52 40.64) (size 0.8) (drill 0.4) (layers F.Cu B.Cu) (net 4))
   (via (at 96.52 38.1) (size 0.8) (drill 0.4) (layers F.Cu B.Cu) (net 4))
-  (segment (start 93.98 40.64) (end 96.52 40.64) (width 0.4) (layer B.Cu) (net 4))
-  (segment (start 96.52 40.64) (end 96.52 38.1) (width 0.4) (layer B.Cu) (net 4))
-  (segment (start 96.52 35.56) (end 96.52 38.1) (width 0.4) (layer B.Cu) (net 4))
-  (segment (start 96.52 35.56) (end 93.98 35.56) (width 0.4) (layer B.Cu) (net 4))
-  (segment (start 93.98 35.56) (end 91.44 35.56) (width 0.4) (layer B.Cu) (net 4))
-  (segment (start 91.44 35.56) (end 88.9 35.56) (width 0.4) (layer B.Cu) (net 4))
-  (segment (start 88.9 35.56) (end 86.36 35.56) (width 0.4) (layer B.Cu) (net 4))
-  (segment (start 86.36 35.56) (end 83.82 35.56) (width 0.4) (layer B.Cu) (net 4))
-  (segment (start 83.82 35.56) (end 71.12 35.56) (width 0.4) (layer B.Cu) (net 4))
-  (segment (start 96.52 40.64) (end 96.52 55.88) (width 0.4) (layer B.Cu) (net 4))
-  (segment (start 96.52 55.88) (end 68.58 55.88) (width 0.4) (layer B.Cu) (net 4))
   (segment (start 68.58 55.88) (end 68.58 55.88) (width 0.4) (layer B.Cu) (net 4))
   (via (at 68.58 55.88) (size 0.8) (drill 0.4) (layers F.Cu B.Cu) (net 4))
-  (segment (start 69.380001 35.56) (end 71.12 35.56) (width 0.4) (layer B.Cu) (net 4))
-  (segment (start 68.58 55.88) (end 68.58 53.34) (width 0.4) (layer B.Cu) (net 4))
-  (segment (start 68.58 53.34) (end 68.58 35.56) (width 0.4) (layer B.Cu) (net 4))
-  (segment (start 68.58 35.56) (end 71.12 35.56) (width 0.4) (layer B.Cu) (net 4))
   (segment (start 88.9 47.83) (end 89.05 47.68) (width 0.25) (layer F.Cu) (net 5))
   (segment (start 88.9 53.34) (end 88.9 47.83) (width 0.25) (layer F.Cu) (net 5))

Commit message: シルク印字を入れる
Other:
- board text added: "2018/08/12 By Akira345"
Changed lines of the file:
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@@
   (general
     (thickness 1.6)
-    (drawings 7)
+    (drawings 9)
     (tracks 50)
     (zones 0)
@@
     )
   )
+  (gr_text "2018/08/12\nBy Akira345" (at 93.98 49.53 90) (layer F.SilkS)
+    (effects (font (size 1.2 1.2) (thickness 0.1)))
+  )
+  (gr_text "2018/08/12\nBy Akira345" (at 93.98 49.53 90) (layer B.SilkS)
+    (effects (font (size 1.2 1.2) (thickness 0.1)) (justify mirror))
+  )
   (gr_line (start 67.31 34.29) (end 97.79 34.29) (layer Edge.Cuts) (width 0.15))
